Commit message: hand to eye calibration

File: hustac_pg_v2/robots/hustac_pg_v2.urdf (robot description, URDF)
Before this commit: robot hustac_pg_v2, 27 links, 26 joints
Joints:
- joint gaze_joint1: limit lower=-6.28 upper=6.28 effort=300 velocity=1 -> lower=-3.14 upper=3.14 effort=300 velocity=1
- joint gaze_joint2: limit lower=-6.28 upper=6.28 effort=300 velocity=1 -> lower=-3.14 upper=3.14 effort=300 velocity=1
- joint left_joint1: limit lower=-6.28 upper=6.28 effort=300 velocity=1 -> lower=-3.14 upper=3.14 effort=300 velocity=1
- joint left_joint2: limit lower=-6.28 upper=6.28 effort=300 velocity=1 -> lower=-3.14 upper=3.14 effort=300 velocity=1
- joint left_joint3: limit lower=-6.28 upper=6.28 effort=300 velocity=1 -> lower=-3.14 upper=3.14 effort=300 velocity=1
- joint left_joint4: limit lower=-6.28 upper=6.28 effort=300 velocity=1 -> lower=-3.14 upper=3.14 effort=300 velocity=1
- joint left_joint5: limit lower=-6.28 upper=6.28 effort=300 velocity=1 -> lower=-3.14 upper=3.14 effort=300 velocity=1
- joint left_joint6: limit lower=-6.28 upper=6.28 effort=300 velocity=1 -> lower=-3.14 upper=3.14 effort=300 velocity=1
- joint left_joint7: limit lower=-6.28 upper=6.28 effort=300 velocity=1 -> lower=-3.14 upper=3.14 effort=300 velocity=1
- joint right_joint1: limit lower=-6.28 upper=6.28 effort=300 velocity=1 -> lower=-3.14 upper=3.14 effort=300 velocity=1
- joint right_joint2: limit lower=-6.28 upper=6.28 effort=300 velocity=1 -> lower=-3.14 upper=3.14 effort=300 velocity=1
- joint right_joint3: limit lower=-6.28 upper=6.28 effort=300 velocity=1 -> lower=-3.14 upper=3.14 effort=300 velocity=1
- joint right_joint4: limit lower=-6.28 upper=6.28 effort=300 velocity=1 -> lower=-3.14 upper=3.14 effort=300 velocity=1
- joint right_joint5: limit lower=-6.28 upper=6.28 effort=300 velocity=1 -> lower=-3.14 upper=3.14 effort=300 velocity=1
- joint right_joint6: limit lower=-6.28 upper=6.28 effort=300 velocity=1 -> lower=-3.14 upper=3.14 effort=300 velocity=1
- joint right_joint7: limit lower=-6.28 upper=6.28 effort=300 velocity=1 -> lower=-3.14 upper=3.14 effort=300 velocity=1

Commit message: upgrade pillow requirements to version 6.2.0

File: hustac_pg_v2/robots/hustac_pg_v2.urdf (robot description, URDF)
Before this commit: robot hustac_pg_v2, 27 links, 26 joints
Joints:
- joint left_ee_joint: origin xyz=-0.0110000000000008 0.0105000000000003 0.0221811953944651 rpy=1.5707963267949 6.40215462385206E-19 2.24264473650599E-16 -> xyz=-0.0110000000000008 0.0105000000000003 0.0221811953944651 rpy=1.570796327 2.35619449 0
- joint left_ee_joint2: origin xyz=0.0110000000000001 0.0105000000000002 0.0221811953944651 rpy=1.5707963267949 6.40215462385206E-19 2.24264473650599E-16 -> xyz=0.0110000000000001 0.0105000000000002 0.0221811953944651 rpy=1.570796327 -2.35619449 0
- joint right_ee_joint: origin xyz=0.0110000000000067 -0.0104999999999925 0.0221811953944649 rpy=1.5707963267949 7.47513322448154E-18 -3.14159265358979 -> xyz=0.0110000000000067 -0.0104999999999925 0.0221811953944649 rpy=1.5707963267949 2.35619449 -3.14159265358979
- joint right_ee_joint2: origin xyz=-0.0110000000000009 -0.0104999999999998 0.0221811953944632 rpy=1.5707963267949 7.47513322448154E-18 -3.14159265358979 -> xyz=-0.0110000000000009 -0.0104999999999998 0.0221811953944632 rpy=1.5707963267949 -2.35619449 -3.14159265358979
